Commit message: made some changes

File: description/depth_camera.xacro (robot description, xacro)
@@ -45,5 +45,5 @@
                 <imageTopicName>image_raw</imageTopicName>
                 <cameraInfoTopicName>camera_info</cameraInfoTopicName>
-                <updateRate>20.0</updateRate>
+                <updateRate>30.0</updateRate>
                 <cameraName>usb_cam</cameraName>
                 <!-- <frameName>/robot_camera_link</frameName> -->

File: description/robot_core.xacro (robot description, xacro)
@@ -464,23 +464,68 @@
         <mu2 value="0.45"/>
     </gazebo> -->
+<!--
     <gazebo reference="left_wheel1">
         <material>Gazebo/Grey</material>
-        <mu1 value="0.1"/>
-        <mu2 value="0.095"/>
+        <mu1 value="0.6"/>
+        <mu2 value="0.595"/>
     </gazebo>
         <gazebo reference="right_wheel1">
         <material>Gazebo/Grey</material>
-        <mu1 value="0.1"/>
-        <mu2 value="0.095"/>
+        <mu1 value="0.6"/>
+        <mu2 value="0.595"/>
     </gazebo>
         <gazebo reference="left_wheel2">
         <material>Gazebo/Grey</material>
-        <mu1 value="0.1"/>
-        <mu2 value="0.095"/>
+        <mu1 value="0.7"/>
+        <mu2 value="0.695"/>
     </gazebo>
         <gazebo reference="right_wheel2">
         <material>Gazebo/Grey</material>
-        <mu1 value="0.1"/>
-        <mu2 value="0.095"/>
-    </gazebo>
+        <mu1 value="0.7"/>
+        <mu2 value="0.95"/>
+    </gazebo>
+    	<gazebo reference="left_wheel3">
+        <material>Gazebo/Grey</material>
+        <mu1 value="0.6"/>
+        <mu2 value="0.595"/>
+    </gazebo>
+        <gazebo reference="right_wheel3">
+        <material>Gazebo/Grey</material>
+        <mu1 value="0.6"/>
+        <mu2 value="0.595"/>
+    </gazebo>
+-->
+<!-- Front Wheels -->
+<gazebo reference="left_wheel1">
+  <material>Gazebo/Grey</material>
+  <mu1 value="0.9"/>
+  <mu2 value="0.1"/>
+</gazebo>
+<gazebo reference="right_wheel1">
+  <material>Gazebo/Grey</material>
+  <mu1 value="0.9"/>
+  <mu2 value="0.1"/>
+</gazebo>
+<!-- Middle Wheels -->
+<gazebo reference="left_wheel2">
+  <material>Gazebo/Grey</material>
+  <mu1 value="1.0"/>
+  <mu2 value="1.0"/>
+</gazebo>
+<gazebo reference="right_wheel2">
+  <material>Gazebo/Grey</material>
+  <mu1 value="1.0"/>
+  <mu2 value="1.0"/>
+</gazebo>
+<!-- Rear Wheels -->
+<gazebo reference="left_wheel3">
+  <material>Gazebo/Grey</material>
+  <mu1 value="0.9"/>
+  <mu2 value="0.1"/>
+</gazebo>
+<gazebo reference="right_wheel3">
+  <material>Gazebo/Grey</material>
+  <mu1 value="0.9"/>
+  <mu2 value="0.1"/>
+</gazebo>
 </robot>
