Commit message: simulation ready rover

File: description/gazebo_control.xacro (robot description, xacro)
@@ -2,20 +2,31 @@
 <robot xmlns:xacro="http://www.ros.org/wiki/xacro">
     <gazebo>
-        <plugin name="diff_drive" filename="libgazebo_ros_diff_drive.so">
-            <!-- Wheel Information -->
-            <left_joint>left_wheel_joint</left_joint>
-            <right_joint>right_wheel_joint</right_joint>
-            <wheel_separation>0.35</wheel_separation>
-            <wheel_diameter>0.1</wheel_diameter>
-            <!-- Limits -->
-            <max_wheel_torque>200</max_wheel_torque>
-            <max_wheel_acceleration>10.0</max_wheel_acceleration>
-            <!-- Output -->
-            <odometry_frame>odom</odometry_frame>
-            <robot_base_frame>base_link</robot_base_frame>
-            <publish_odom>true</publish_odom>
-            <publish_odom_tf>true</publish_odom_tf>
-            <publish_wheel_tf>true</publish_wheel_tf>
-        </plugin>
+        <!-- <plugin name="JointStatePublisher" filename="libJointStatePublisher.so"/> -->
+        <plugin name='diff_drive' filename='libgazebo_ros_diff_drive.so'>
+        <!-- <ros> -->
+          <!-- <namespace>/demo</namespace> -->
+          <!-- <remapping>cmd_vel:</remapping> -->
+          <!-- <remapping>odom:=odom_demo</remapping> -->
+        <!-- </ros> -->
+        <!-- wheels -->
+         <num_wheel_pairs>3</num_wheel_pairs>
+            <left_joint>front_left_wheel_joint</left_joint>
+            <left_joint>middle_left_wheel_joint</left_joint>
+            <left_joint>rear_right_wheel_joint</left_joint>
+            <right_joint>front_right_wheel_joint</right_joint>
+            <right_joint>middle_right_wheel_joint</right_joint>
+            <right_joint>rear_left_wheel_joint</right_joint>
+        <!-- kinematics -->
+        <wheel_separation>0.43</wheel_separation>
+        <wheel_diameter>0.156</wheel_diameter>
+        <!-- limits -->
+        <max_wheel_torque>20</max_wheel_torque>
+        <max_wheel_acceleration>1.0</max_wheel_acceleration>
+        <!-- output -->
+        <!-- <publish_odom>true</publish_odom>
+        <publish_odom_tf>true</publish_odom_tf>
+        <publish_wheel_tf>false</publish_wheel_tf>
+        <robot_base_frame>base_footprint</robot_base_frame> -->
+      </plugin>
     </gazebo>
 </robot>

File: description/lidar.xacro (robot description, xacro)
@@ -4,35 +4,28 @@
         <parent link="chassis"/>
         <child link="laser_frame"/>
-        <origin xyz="0.122 0 0.212" rpy="0 0 0"/>
+        <origin xyz="0.035 0 0.095" rpy="0 0 0"/>
     </joint>
     <link name="laser_frame">
         <visual>
             <geometry>
-                <cylinder radius="0.05" length="0.04"/>
+                <cylinder radius="0.035" length="0.02"/>
             </geometry>
-            <material name="black"/>
-        </visual>
-        <visual>
-            <origin xyz="0 0 -0.05"/>
-            <geometry>
-                <cylinder radius="0.01" length="0.1"/>
-            </geometry>
-            <material name="black"/>
+            <material name="red"/>
         </visual>
         <collision>
             <geometry>
-                <cylinder radius="0.05" length="0.04"/>
+                <cylinder radius="0.035" length="0.02"/>
             </geometry>
         </collision>
-        <xacro:inertial_cylinder mass="0.1" length="0.04" radius="0.05">
+        <xacro:inertial_cylinder mass="0.1" length="0.02" radius="0.035">
             <origin xyz="0 0 0" rpy="0 0 0"/>
         </xacro:inertial_cylinder>
     </link>
     <gazebo reference="laser_frame">
-        <material>Gazebo/Black</material>
+        <material>Gazebo/Red</material>
         <sensor name="laser" type="ray">
             <pose> 0 0 0 0 0 0 </pose>
             <visualize>true</visualize>
-            <update_rate>30</update_rate>
+            <update_rate>10</update_rate>
             <ray>
                 <scan>
@@ -45,10 +38,10 @@
                 <range>
                     <min>0.3</min>
-                    <max>25</max>
+                    <max>12</max>
                 </range>
             </ray>
             <plugin name="laser_controller" filename="libgazebo_ros_ray_sensor.so">
                 <ros>
-                    <argument>~/out:=scan</argument>
+                     <argument>-ros-args --remap ~/out:=sca</argument>
                 </ros>
                 <output_type>sensor_msgs/LaserScan</output_type>

File: description/robot.urdf.xacro (robot description, xacro)
@@ -1,6 +1,15 @@
 <?xml version="1.0"?>
 <robot xmlns:xacro="http://www.ros.org/wiki/xacro"  name="robot">
+    <!-- <xacro:arg name="use_ros2_control" default="true"/>
+    <xacro:arg name="sim_mode" default="false"/> -->
     <xacro:include filename="robot_core.xacro" />
-    <xacro:include filename="lidar.xacro" />
-    <xacro:include filename="ros2_control.xacro" />
+    <xacro:include filename="gazebo_control.xacro" />
+    <xacro:include filename="depth_camera.xacro" />
+    <xacro:include filename="imu.xacro" />
+    <!-- <xacro:if value="$(arg use_ros2_control)">
+        <xacro:include filename="ros2_control.xacro" />
+    </xacro:if>
+    <xacro:unless value="$(arg use_ros2_control)">
+    </xacro:unless>
+    <xacro:include filename="depth_camera.xacro" /> -->
 </robot>

File: description/robot_core.xacro (robot description, xacro)
@@ -22,9 +22,9 @@
  <!-- BASEFOOTPRINT LINK -->
     <joint name="base_footprint_joint" type="fixed">
-        <parent link="base_link"/>
-        <child link="base_footprint"/>
+        <parent link="base_footprint"/>
+        <child link="base_link"/>
         <origin xyz="0 0 0 " rpy="0 0 0"/>
     </joint>
-  <link name="base_footprint">
+    <link name="base_footprint">
     </link>
     <!-- CHASSIS LINK -->
@@ -32,22 +32,22 @@
         <parent link="base_link"/>
         <child link="chassis"/>
-        <origin xyz="-0.025 0 0"/>
+        <origin xyz="0 0 0"/>
     </joint>
     <link name="chassis">
         <visual>
-            <origin xyz="0.09 0 0.035"/>
-            <geometry>
-                <box size="0.18 0.18 0.07"/>
-            </geometry>
-            <material name="white"/>
-        </visual>
-        <collision>
-            <origin xyz="0.15 0 0.075"/>
-            <geometry>
-                <box size="0.3 0.3 0.15"/>
-            </geometry>
-        </collision>
-        <xacro:inertial_box mass="0.5" x="0.3" y="0.3" z="0.15">
-            <origin xyz="0.15 0 0.075" rpy="0 0 0"/>
+            <geometry>
+                <box size="0.6 0.4 0.2"/>
+            </geometry>
+            <origin xyz="0 0 0" rpy="0 0 0"/>
+            <material name="blue"/>
+        </visual>
+        <collision>
+            <geometry>
+                <box size="0.6 0.4 0.2"/>
+            </geometry>
+            <origin xyz="0 0 0" rpy="0 0 0"/>
+        </collision>
+        <xacro:inertial_box mass="1" x="0.6" y="0.4" z="0.2">
+            <origin xyz="0 0 0" rpy="0 0 0"/>
         </xacro:inertial_box>
     </link>
@@ -55,81 +55,432 @@
         <material>Gazebo/White</material>
     </gazebo>
-    <!-- LEFT WHEEL LINK -->
-    <joint name="left_wheel_joint" type="continuous">
+    <link name="left_diff_link" />
+    <joint name="left_diff_joint" type="fixed">
         <parent link="base_link"/>
-        <child link="left_wheel"/>
-        <origin xyz="0 0.105 0" rpy="-${pi/2} 0 0" />
-        <axis xyz="0 0 1"/>
-    </joint>
-    <link name="left_wheel">
-        <visual>
-            <geometry>
-                <cylinder radius="0.03" length="0.025"/>
-            </geometry>
-            <material name="blue"/>
-        </visual>
-        <collision>
-            <geometry>
-                <cylinder radius="0.03" length="0.025"/>
-            </geometry>
-        </collision>
-        <xacro:inertial_cylinder mass="0.1" length="0.025" radius="0.03">
-            <origin xyz="0 0 0" rpy="0 0 0"/>
-        </xacro:inertial_cylinder>
-    </link>
-    <gazebo reference="left_wheel">
-        <material>Gazebo/Blue</material>
-    </gazebo>
-    <joint name="right_wheel_joint" type="continuous">
+        <child link="left_diff_link"/>
+        <axis xyz="0 0 1"/>
+        <origin rpy="-${pi/2} 0 0" xyz="0 0.215 0"/>
+        <limit lower="-3.14" upper="3.14" effort="10" velocity="1"/>
+    </joint>
+    <link name="l_rod_1">
+        <visual>
+            <geometry>
+                <box size="0.03 0.03 0.64"/>
+            </geometry>
+            <material name="red"/>
+            <origin xyz="0 0 -0.32" rpy="0 0 0"/>
+        </visual>
+        <collision>
+            <geometry>
+                <box size="0.03 0.03 0.64"/>
+            </geometry>
+            <material name="red"/>
+            <origin xyz="0 0 -0.32" rpy="0 0 0"/>
+        </collision>
+        <xacro:inertial_box mass="0.5" x="0.03" y="0.03" z="0.64">
+            <origin xyz="0 0 -0.32" rpy="0 0 0"/>
+        </xacro:inertial_box>
+    </link>
+    <link name="l_rod_2">
+        <visual>
+            <geometry>
+                <box size="0.03 0.03 0.28"/>
+            </geometry>
+            <material name="red"/>
+            <origin xyz="0 0 -0.14" rpy="0 0 0"/>
+        </visual>
+        <collision>
+            <geometry>
+                <box size="0.03 0.03 0.28"/>
+            </geometry>
+            <material name="red"/>
+            <origin xyz="0 0 -0.14" rpy="0 0 0"/>
+        </collision>
+        <xacro:inertial_box mass="0.5" x="0.03" y="0.03" z="0.28">
+            <origin xyz="0 0 -0.14" rpy="0 0 0"/>
+        </xacro:inertial_box>
+    </link>
+    <link name="left_rod2_sub_link" />
+    <link name="l_rod_3">
+        <visual>
+            <geometry>
+                <box size="0.03 0.03 0.36"/>
+            </geometry>
+            <material name="red"/>
+            <origin xyz="0 0 -0.18" rpy="0 0 0"/>
+        </visual>
+        <collision>
+            <geometry>
+                <box size="0.03 0.03 0.36"/>
+            </geometry>
+            <material name="red"/>
+            <origin xyz="0 0 -0.18" rpy="0 0 0"/>
+        </collision>
+        <xacro:inertial_box mass="0.5" x="0.03" y="0.03" z="0.36">
+            <origin xyz="0 0 -0.18" rpy="0 0 0"/>
+        </xacro:inertial_box>
+    </link>
+    <link name="l_rod_4">
+        <visual>
+            <geometry>
+                <box size="0.03 0.03 0.36"/>
+            </geometry>
+            <material name="red"/>
+            <origin xyz="0 0 -0.18" rpy="0 0 0"/>
+        </visual>
+        <collision>
+            <geometry>
+                <box size="0.03 0.03 0.36"/>
+            </geometry>
+            <material name="red"/>
+            <origin xyz="0 0 -0.18" rpy="0 0 0"/>
+        </collision>
+        <xacro:inertial_box mass="0.5" x="0.03" y="0.03" z="0.36">
+            <origin xyz="0 0 -0.18" rpy="0 0 0"/>
+        </xacro:inertial_box>
+    </link>
+    <joint name="left_diff_rod1" type="fixed">
+        <parent link="left_diff_link"/>
+        <child link="l_rod_1"/>
+        <axis xyz="0 0 1"/>
+        <origin rpy="${pi/2} 0 -0.895" xyz="0 0 0"/>
+    </joint>
+    <joint name="left_diff_rod2" type="fixed">
+        <parent link="left_diff_link"/>
+        <child link="l_rod_2"/>
+        <axis xyz="0 0 1"/>
+        <origin rpy="${pi/2} 0 0.785" xyz="0 0 0"/>
+    </joint>
+    <joint name="left_rod2_sub_rod1_joint" type="fixed">
+        <parent link="left_rod2_sub_link"/>
+        <child link="l_rod_3"/>
+        <origin rpy="${pi/2} 0 0" xyz="0 0 0"/>
+    </joint>
+    <joint name="left_rod2_sub_joint" type="continuous">
+        <parent link="l_rod_2"/>
+        <child link="left_rod2_sub_link"/>
+        <axis xyz="0 0 1"/>
+        <origin rpy="-${pi/2} 0 0" xyz="0 0 -0.28"/>
+        <limit lower="-3.14" upper="3.14" effort="10" velocity="1"/>
+    </joint>
+    <joint name="left_rod2_sub_rod2_joint" type="fixed">
+        <parent link="left_rod2_sub_link"/>
+        <child link="l_rod_4"/>
+        <origin rpy="${pi/2} 0 -1.588" xyz="0 0 0"/>
+    </joint>
+    <link name="right_diff_link" />
+    <link name="r_rod_1">
+        <visual>
+            <geometry>
+                <box size="0.03 0.03 0.64"/>
+            </geometry>
+            <material name="red"/>
+            <origin xyz="0 0 -0.32" rpy="0 0 0"/>
+        </visual>
+        <collision>
+            <geometry>
+                <box size="0.03 0.03 0.64"/>
+            </geometry>
+            <material name="red"/>
+            <origin xyz="0 0 -0.32" rpy="0 0 0"/>
+        </collision>
+        <xacro:inertial_box mass="0.5" x="0.03" y="0.03" z="0.64">
+            <origin xyz="0 0 -0.32" rpy="0 0 0"/>
+        </xacro:inertial_box>
+    </link>
+    <link name="r_rod_2">
+        <visual>
+            <geometry>
+                <box size="0.03 0.03 0.28"/>
+            </geometry>
+            <material name="red"/>
+            <origin xyz="0 0 -0.14" rpy="0 0 0"/>
+        </visual>
+        <collision>
+            <geometry>
+                <box size="0.03 0.03 0.28"/>
+            </geometry>
+            <material name="red"/>
+            <origin xyz="0 0 -0.14" rpy="0 0 0"/>
+        </collision>
+        <xacro:inertial_box mass="0.5" x="0.03" y="0.03" z="0.28">
+            <origin xyz="0 0 -0.14" rpy="0 0 0"/>
+        </xacro:inertial_box>
+    </link>
+    <link name="right_rod2_sub_link" />
+    <link name="r_rod_3">
+        <visual>
+            <geometry>
+                <box size="0.03 0.03 0.36"/>
+            </geometry>
+            <material name="red"/>
+            <origin xyz="0 0 -0.18" rpy="0 0 0"/>
+        </visual>
+        <collision>
+            <geometry>
+                <box size="0.03 0.03 0.36"/>
+            </geometry>
+            <material name="red"/>
+            <origin xyz="0 0 -0.18" rpy="0 0 0"/>
+        </collision>
+        <xacro:inertial_box mass="0.5" x="0.03" y="0.03" z="0.36">
+            <origin xyz="0 0 -0.18" rpy="0 0 0"/>
+        </xacro:inertial_box>
+    </link>
+    <link name="r_rod_4">
+        <visual>
+            <geometry>
+                <box size="0.03 0.03 0.36"/>
+            </geometry>
+            <material name="red"/>
+            <origin xyz="0 0 -0.18" rpy="0 0 0"/>
+        </visual>
+        <collision>
+            <geometry>
+                <box size="0.03 0.03 0.36"/>
+            </geometry>
+            <material name="red"/>
+            <origin xyz="0 0 -0.18" rpy="0 0 0"/>
+        </collision>
+        <xacro:inertial_box mass="0.5" x="0.03" y="0.03" z="0.36">
+            <origin xyz="0 0 -0.18" rpy="0 0 0"/>
+        </xacro:inertial_box>
+    </link>
+    <joint name="right_diff_joint" type="fixed">
         <parent link="base_link"/>
-        <child link="right_wheel"/>
-        <origin xyz="0 -0.105 0" rpy="${pi/2} 0 0" />
+        <child link="right_diff_link"/>
+        <axis xyz="0 0 1"/>
+        <origin rpy="-${pi/2} 0 0" xyz="0 -0.215 0"/>
+        <limit lower="-3.14" upper="3.14" effort="10" velocity="1"/>
+    </joint>
+    <joint name="right_diff_rod1" type="fixed">
+        <parent link="right_diff_link"/>
+        <child link="r_rod_1"/>
+        <axis xyz="0 0 1"/>
+        <origin rpy="${pi/2} 0 -0.895" xyz="0 0 0"/>
+    </joint>
+    <joint name="right_diff_rod2" type="fixed">
+        <parent link="right_diff_link"/>
+        <child link="r_rod_2"/>
+        <axis xyz="0 0 1"/>
+        <origin rpy="${pi/2} 0 0.785" xyz="0 0 0"/>
+    </joint>
+    <joint name="right_rod2_sub_joint" type="continuous">
+        <parent link="r_rod_2"/>
+        <child link="right_rod2_sub_link"/>
+        <axis xyz="0 0 1"/>
+        <origin rpy="-${pi/2} 0 0" xyz="0 0 -0.28"/>
+        <limit lower="-3.14" upper="3.14" effort="10" velocity="1"/>
+    </joint>
+    <joint name="right_rod2_sub_rod1_joint" type="fixed">
+        <parent link="right_rod2_sub_link"/>
+        <child link="r_rod_3"/>
+        <origin rpy="${pi/2} 0 0" xyz="0 0 0"/>
+    </joint>
+    <joint name="right_rod2_sub_rod2_joint" type="fixed">
+        <parent link="right_rod2_sub_link"/>
+        <child link="r_rod_4"/>
+        <origin rpy="${pi/2} 0 -1.588" xyz="0 0 0"/>
+    </joint>
+   <link name="left_wheel1">
+        <visual>
+            <geometry>
+                <cylinder radius="0.078" length="0.075"/>
+            </geometry>
+            <origin xyz="0 0 0.0525" rpy="0 0 0"/>
+            <material name="white"/>
+        </visual>
+        <collision>
+            <geometry>
+                <cylinder radius="0.078" length="0.075"/>
+            </geometry>
+            <origin xyz="0 0 0.0525" rpy="0 0 0"/>
+            <material name="white"/>
+        </collision>
+        <xacro:inertial_cylinder mass="0.5" radius="0.078" length="0.075" >
+            <origin xyz="0 0 0.0525" rpy="0 0 0"/>
+        </xacro:inertial_cylinder>
+    </link>
+    <link name="left_wheel2">
+        <visual>
+            <geometry>
+                <cylinder radius="0.078" length="0.075"/>
+            </geometry>
+            <origin xyz="0 0 0.0525" rpy="0 0 0"/>
+            <material name="white"/>
+        </visual>
+        <collision>
+            <geometry>
+                <cylinder radius="0.078" length="0.075"/>
+            </geometry>
+            <origin xyz="0 0 0.0525" rpy="0 0 0"/>
+            <material name="white"/>
+        </collision>
+        <xacro:inertial_cylinder mass="0.5" radius="0.078" length="0.075" >
+            <origin xyz="0 0 0.0525" rpy="0 0 0"/>
+        </xacro:inertial_cylinder>
+    </link>
+    <link name="left_wheel3">
+        <visual>
+            <geometry>
+                <cylinder radius="0.078" length="0.075"/>
+            </geometry>
+            <origin xyz="0 0 0.0525" rpy="0 0 0"/>
+            <material name="white"/>
+        </visual>
+        <collision>
+            <geometry>
+                <cylinder radius="0.078" length="0.075"/>
+            </geometry>
+            <origin xyz="0 0 0.0525" rpy="0 0 0"/>
+            <material name="white"/>
+        </collision>
+        <xacro:inertial_cylinder mass="0.5" radius="0.078" length="0.075" >
+            <origin xyz="0 0 0.0525" rpy="0 0 0"/>
+        </xacro:inertial_cylinder>
+    </link>
+    <link name="right_wheel1">
+        <visual>
+            <geometry>
+                <cylinder radius="0.078" length="0.075"/>
+            </geometry>
+            <origin xyz="0 0 0.0525" rpy="0 0 0"/>
+            <material name="white"/>
+        </visual>
+        <collision>
+            <geometry>
+                <cylinder radius="0.078" length="0.075"/>
+            </geometry>
+            <origin xyz="0 0 0.0525" rpy="0 0 0"/>
+            <material name="white"/>
+        </collision>
+        <xacro:inertial_cylinder mass="0.5" radius="0.078" length="0.075" >
+            <origin xyz="0 0 0.0525" rpy="0 0 0"/>
+        </xacro:inertial_cylinder>
+    </link>
+    <link name="right_wheel2">
+        <visual>
+            <geometry>
+                <cylinder radius="0.078" length="0.075"/>
+            </geometry>
+            <origin xyz="0 0 0.0525" rpy="0 0 0"/>
+            <material name="white"/>
+        </visual>
+        <collision>
+            <geometry>
+                <cylinder radius="0.078" length="0.075"/>
+            </geometry>
+            <origin xyz="0 0 0.0525" rpy="0 0 0"/>
+            <material name="white"/>
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
File: description/ros2_control.xacro (robot description, xacro)
@@ -1,9 +1,37 @@
 <?xml version="1.0"?>
 <robot xmlns:xacro="http://www.ros.org/wiki/xacro">
-    <ros2_control name="GazeboSystem" type="system">
-        <hardware>
+<!--     <ros2_control name="GazeboSystem" type="system">
+           <hardware>
             <plugin>gazebo_ros2_control/GazeboSystem</plugin>
-        </hardware>
-        <joint name="left_wheel_joint">
+           </hardware>
+           <joint name="left_wheel_joint">
+            <command_interface name="velocity">
+                <param name="min">-10</param>
+                <param name="max">10</param>
+            </command_interface>
+            <state_interface name="velocity"/>
+            <state_interface name="position"/>
+        </joint>
+        <joint name="right_wheel_joint">
+            <command_interface name="velocity">
+                <param name="min">-10</param>
+                <param name="max">10</param>
+            </command_interface>
+            <state_interface name="velocity"/>
+            <state_interface name="position"/>
+        </joint>
+    </ros2_control> -->
+     <ros2_control name="realBot" type="system">
+           <hardware>
+            <plugin>diffdrive_arduino/DiffDriveArduino</plugin>
+            <param name="left_wheel_name">left_wheel_joint</param>
+            <param name="right_wheel_name">right_wheel_joint</param>
+            <param name="loop_rate">30</param>
+            <param name="device">/dev/ttyACM0</param>
+            <param name="baud_rate">57600</param>
+            <param name="timeout">1000</param>
+            <param name="enc_counts_per_rev">294</param>
+           </hardware>
+           <joint name="left_wheel_joint">
             <command_interface name="velocity">
                 <param name="min">-10</param>
@@ -22,8 +50,8 @@
         </joint>
     </ros2_control>
-    <gazebo>
-        <plugin name="gazebo_ros2_control" filename="libgazebo_ros2_control.so">
+      <gazebo>
+          <plugin name="gazebo_ros2_control" filename="libgazebo_ros2_control.so">
             <parameters>$(find Test_bot)/config/my_controllers.yaml</parameters>
-        </plugin>
-    </gazebo>
+          </plugin>
+      </gazebo>
 </robot>
