Commit message: added rtab launch

File: description/gazebo_control.xacro (robot description, xacro)
@@ -22,5 +22,5 @@
         <!-- limits -->
         <max_wheel_torque>30</max_wheel_torque>
-        <max_wheel_acceleration>1.0</max_wheel_acceleration>
+        <max_wheel_acceleration>10</max_wheel_acceleration>
         <!-- output -->
         <!-- <publish_odom>true</publish_odom>

File: description/robot_core.xacro (robot description, xacro)
@@ -433,35 +433,24 @@
         <origin xyz="0.49 0.215 -0.4117" rpy="-${pi/2} 0 0"/>
    </joint>
-<!--
-    <gazebo reference="left_wheel3">
-        <material>Gazebo/Grey</material>
-        <mu1 value="0.5"/>
-        <mu2 value="0.45"/>
-    </gazebo>
     <gazebo reference="left_wheel2">
         <material>Gazebo/Grey</material>
-        <mu1 value="0.5"/>
-        <mu2 value="0.45"/>
+        <mu1 value="0.2"/>
+        <mu2 value="0.195"/>
     </gazebo>
     <gazebo reference="left_wheel1">
         <material>Gazebo/Grey</material>
-        <mu1 value="0.5"/>
-        <mu2 value="0.45"/>
-    </gazebo>
-    <gazebo reference="right_wheel3">
-        <material>Gazebo/Grey</material>
-        <mu1 value="0.5"/>
-        <mu2 value="0.45"/>
+        <mu1 value="0.1"/>
+        <mu2 value="0.095"/>
     </gazebo>
     <gazebo reference="right_wheel2">
         <material>Gazebo/Grey</material>
-        <mu1 value="0.5"/>
-        <mu2 value="0.45"/>
+        <mu1 value="0.2"/>
+        <mu2 value="0.195"/>
     </gazebo>
     <gazebo reference="right_wheel1">
         <material>Gazebo/Grey</material>
-        <mu1 value="0.5"/>
-        <mu2 value="0.45"/>
-    </gazebo> -->
+        <mu1 value="0.1"/>
+        <mu2 value="0.095"/>
+    </gazebo>
 <!--
     <gazebo reference="left_wheel1">
@@ -496,5 +485,5 @@
     </gazebo>
 -->
-<!-- Front Wheels -->
+<!--
 <gazebo reference="left_wheel1">
   <material>Gazebo/Grey</material>
@@ -507,5 +496,4 @@
   <mu2 value="0.1"/>
 </gazebo>
-<!-- Middle Wheels -->
 <gazebo reference="left_wheel2">
   <material>Gazebo/Grey</material>
@@ -518,5 +506,4 @@
   <mu2 value="1.0"/>
 </gazebo>
-<!-- Rear Wheels -->
 <gazebo reference="left_wheel3">
   <material>Gazebo/Grey</material>
@@ -528,4 +515,4 @@
   <mu1 value="0.9"/>
   <mu2 value="0.1"/>
-</gazebo>
+</gazebo> -->
 </robot>
